File: hw/sensor/sensor.kicad_pcb (KiCad board)
At the start: 2 copper layers, 75.1 x 14 mm, 4 parts, among them X1 TestPoint_Pad_2.0x2.0mm, X2 TestPoint_Pad_2.0x2.0mm, X3 TestPoint_Pad_2.0x2.0mm, X4 TestPoint_Pad_2.0x2.0mm

Commit message: wip
Parts:
- added X5: TestPoint_Pad_2.0x2.0mm, TestPoint:TestPoint_Pad_2.0x2.0mm, F.Cu at (100.0, 81.5)
- added X6: TestPoint_Pad_2.0x2.0mm, TestPoint:TestPoint_Pad_2.0x2.0mm, B.Cu at (100.0, 81.5)
- X2: moved to B.Cu
- X3: moved to F.Cu
- moved X2 11.0 mm to (100.0, 68.5), turned to 90 degrees
- moved X3 11.0 mm to (100.0, 79.5), turned to 270 degrees
Connections:
- X2 pad 1: /CAP2 -> /CAP1
- X3 pad 1: /CAP1 -> /CAP2
Routing:
- net /CAP2: vias 4 -> 8
Other:
- board size 75.1 x 14 mm -> 75.1 x 16 mm
Changed lines of the file:
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@@
   (general
     (thickness 1.6)
-    (drawings 19)
-    (tracks 8)
+    (drawings 21)
+    (tracks 12)
     (zones 0)
-    (modules 4)
+    (modules 6)
     (nets 3)
   )
@@
     (solder_mask_min_width 0.25)
     (aux_axis_origin 0 0)
-    (grid_origin 100 81)
+    (grid_origin 100 74)
     (visible_elements 7FFFFFFF)
     (pcbplotparams
@@
   )
   (module TestPoint:TestPoint_Pad_2.0x2.0mm (layer B.Cu)
-    (at 100 79.5 90)
-    (descr "SMD rectangular pad as test Point, square 2.0mm side length")
-    (tags "test point SMD pad rectangle square")
-    (attr virtual)
-    (fp_text reference X4 (at 0 1.998 -90) (layer B.SilkS)
+    (at 100 81.5 90)
+    (descr "SMD rectangular pad as test Point, square 2.0mm side length")
+    (tags "test point SMD pad rectangle square")
+    (attr virtual)
+    (fp_text reference X6 (at 0 1.998 -90) (layer B.SilkS)
       (effects (font (size 1 1) (thickness 0.15)) (justify mirror))
     )
@@
       (net 2 /CAP2))
   )
-  (module TestPoint:TestPoint_Pad_2.0x2.0mm (layer B.Cu)
-    (at 100 68.5 90)
-    (descr "SMD rectangular pad as test Point, square 2.0mm side length")
-    (tags "test point SMD pad rectangle square")
-    (attr virtual)
-    (fp_text reference X3 (at 0 1.998 90) (layer B.SilkS)
-      (effects (font (size 1 1) (thickness 0.15)) (justify mirror))
-    )
-    (fp_text value TestPoint_Pad_2.0x2.0mm (at 0 -2.05 90) (layer B.Fab)
-      (effects (font (size 1 1) (thickness 0.15)) (justify mirror))
-    )
-    (fp_line (start 1.5 -1.5) (end -1.5 -1.5) (layer B.CrtYd) (width 0.05))
-    (fp_line (start 1.5 -1.5) (end 1.5 1.5) (layer B.CrtYd) (width 0.05))
-    (fp_line (start -1.5 1.5) (end -1.5 -1.5) (layer B.CrtYd) (width 0.05))
-    (fp_line (start -1.5 1.5) (end 1.5 1.5) (layer B.CrtYd) (width 0.05))
-    (fp_line (start -1.2 -1.2) (end -1.2 1.2) (layer B.SilkS) (width 0.12))
-    (fp_line (start 1.2 -1.2) (end -1.2 -1.2) (layer B.SilkS) (width 0.12))
-    (fp_line (start 1.2 1.2) (end 1.2 -1.2) (layer B.SilkS) (width 0.12))
-    (fp_line (start -1.2 1.2) (end 1.2 1.2) (layer B.SilkS) (width 0.12))
-    (fp_text user %R (at 0 2 90) (layer B.Fab)
-      (effects (font (size 1 1) (thickness 0.15)) (justify mirror))
-    )
-    (pad 1 smd rect (at 0 0 90) (size 2 2) (layers B.Cu B.Mask)
-      (net 1 /CAP1))
-  )
   (module TestPoint:TestPoint_Pad_2.0x2.0mm (layer F.Cu)
-    (at 100 79.5 270)
-    (descr "SMD rectangular pad as test Point, square 2.0mm side length")
-    (tags "test point SMD pad rectangle square")
-    (attr virtual)
-    (fp_text reference X2 (at 0 -1.998 90) (layer F.SilkS)
+    (at 100 81.5 270)
+    (descr "SMD rectangular pad as test Point, square 2.0mm side length")
+    (tags "test point SMD pad rectangle square")
+    (attr virtual)
+    (fp_text reference X5 (at 0 -1.998 90) (layer F.SilkS)
       (effects (font (size 1 1) (thickness 0.15)))
     )
@@
       (net 2 /CAP2))
   )
+  (module TestPoint:TestPoint_Pad_2.0x2.0mm (layer B.Cu)
+    (at 100 79.5 90)
+    (descr "SMD rectangular pad as test Point, square 2.0mm side length")
+    (tags "test point SMD pad rectangle square")
+    (attr virtual)
+    (fp_text reference X4 (at 0 1.998 -90) (layer B.SilkS)
+      (effects (font (size 1 1) (thickness 0.15)) (justify mirror))
+    )
+    (fp_text value TestPoint_Pad_2.0x2.0mm (at 0 -2.05 -90) (layer B.Fab)
+      (effects (font (size 1 1) (thickness 0.15)) (justify mirror))
+    )
+    (fp_line (start 1.5 -1.5) (end -1.5 -1.5) (layer B.CrtYd) (width 0.05))
+    (fp_line (start 1.5 -1.5) (end 1.5 1.5) (layer B.CrtYd) (width 0.05))
+    (fp_line (start -1.5 1.5) (end -1.5 -1.5) (layer B.CrtYd) (width 0.05))
+    (fp_line (start -1.5 1.5) (end 1.5 1.5) (layer B.CrtYd) (width 0.05))
+    (fp_line (start -1.2 -1.2) (end -1.2 1.2) (layer B.SilkS) (width 0.12))
+    (fp_line (start 1.2 -1.2) (end -1.2 -1.2) (layer B.SilkS) (width 0.12))
+    (fp_line (start 1.2 1.2) (end 1.2 -1.2) (layer B.SilkS) (width 0.12))
+    (fp_line (start -1.2 1.2) (end 1.2 1.2) (layer B.SilkS) (width 0.12))
+    (fp_text user %R (at 0 2 -90) (layer B.Fab)
+      (effects (font (size 1 1) (thickness 0.15)) (justify mirror))
+    )
+    (pad 1 smd rect (at 0 0 90) (size 2 2) (layers B.Cu B.Mask)
+      (net 2 /CAP2))
+  )
+  (module TestPoint:TestPoint_Pad_2.0x2.0mm (layer F.Cu)
+    (at 100 79.5 270)
+    (descr "SMD rectangular pad as test Point, square 2.0mm side length")
+    (tags "test point SMD pad rectangle square")
+    (attr virtual)
+    (fp_text reference X3 (at 0 -1.998 270) (layer F.SilkS)
+      (effects (font (size 1 1) (thickness 0.15)))
+    )
+    (fp_text value TestPoint_Pad_2.0x2.0mm (at 0 2.05 270) (layer F.Fab)
+      (effects (font (size 1 1) (thickness 0.15)))
+    )
+    (fp_line (start 1.5 1.5) (end -1.5 1.5) (layer F.CrtYd) (width 0.05))
+    (fp_line (start 1.5 1.5) (end 1.5 -1.5) (layer F.CrtYd) (width 0.05))
+    (fp_line (start -1.5 -1.5) (end -1.5 1.5) (layer F.CrtYd) (width 0.05))
+    (fp_line (start -1.5 -1.5) (end 1.5 -1.5) (layer F.CrtYd) (width 0.05))
+    (fp_line (start -1.2 1.2) (end -1.2 -1.2) (layer F.SilkS) (width 0.12))
+    (fp_line (start 1.2 1.2) (end -1.2 1.2) (layer F.SilkS) (width 0.12))
+    (fp_line (start 1.2 -1.2) (end 1.2 1.2) (layer F.SilkS) (width 0.12))
+    (fp_line (start -1.2 -1.2) (end 1.2 -1.2) (layer F.SilkS) (width 0.12))
+    (fp_text user %R (at 0 -2 270) (layer F.Fab)
+      (effects (font (size 1 1) (thickness 0.15)))
+    )
+    (pad 1 smd rect (at 0 0 270) (size 2 2) (layers F.Cu F.Mask)
+      (net 2 /CAP2))
+  )
+  (module TestPoint:TestPoint_Pad_2.0x2.0mm (layer B.Cu)
+    (at 100 68.5 90)
+    (descr "SMD rectangular pad as test Point, square 2.0mm side length")
+    (tags "test point SMD pad rectangle square")
+    (attr virtual)
+    (fp_text reference X2 (at 0 1.998 270) (layer B.SilkS)
+      (effects (font (size 1 1) (thickness 0.15)) (justify mirror))
+    )
+    (fp_text value TestPoint_Pad_2.0x2.0mm (at 0 -2.05 270) (layer B.Fab)
+      (effects (font (size 1 1) (thickness 0.15)) (justify mirror))
+    )
+    (fp_line (start 1.5 -1.5) (end -1.5 -1.5) (layer B.CrtYd) (width 0.05))
+    (fp_line (start 1.5 -1.5) (end 1.5 1.5) (layer B.CrtYd) (width 0.05))
+    (fp_line (start -1.5 1.5) (end -1.5 -1.5) (layer B.CrtYd) (width 0.05))
+    (fp_line (start -1.5 1.5) (end 1.5 1.5) (layer B.CrtYd) (width 0.05))
+    (fp_line (start -1.2 -1.2) (end -1.2 1.2) (layer B.SilkS) (width 0.12))
+    (fp_line (start 1.2 -1.2) (end -1.2 -1.2) (layer B.SilkS) (width 0.12))
+    (fp_line (start 1.2 1.2) (end 1.2 -1.2) (layer B.SilkS) (width 0.12))
+    (fp_line (start -1.2 1.2) (end 1.2 1.2) (layer B.SilkS) (width 0.12))
+    (fp_text user %R (at 0 2 270) (layer B.Fab)
+      (effects (font (size 1 1) (thickness 0.15)) (justify mirror))
+    )
+    (pad 1 smd rect (at 0 0 90) (size 2 2) (layers B.Cu B.Mask)
+      (net 1 /CAP1))
+  )
   (module TestPoint:TestPoint_Pad_2.0x2.0mm (layer F.Cu)
     (at 100 68.5 270)
@@
       (net 1 /CAP1))
   )
+  (gr_line (start 103.5 83) (end 106.5 81) (layer Edge.Cuts) (width 0.05))
+  (gr_line (start 101.5 83) (end 103.5 83) (layer Edge.Cuts) (width 0.05))
   (gr_text "Capacitive sensor ~~1pF\n\n©Projektanker" (at 132.5 74) (layer F.SilkS)
     (effects (font (size 1 1) (thickness 0.15)))
@@
   (gr_line (start 101.5 78) (end 101.5 76) (layer Edge.Cuts) (width 0.05))
   (gr_line (start 100 78) (end 101.5 78) (layer Edge.Cuts) (width 0.05))
-  (gr_line (start 98.5 81) (end 100 81) (layer Edge.Cuts) (width 0.05))
-  (gr_line (start 98.5 78) (end 98.5 81) (layer Edge.Cuts) (width 0.05))
+  (gr_line (start 98.5 83) (end 101.5 83) (layer Edge.Cuts) (width 0.05))
+  (gr_line (start 98.5 78) (end 98.5 83) (layer Edge.Cuts) (width 0.05))
   (gr_line (start 100 78) (end 98.5 78) (layer Edge.Cuts) (width 0.05))
   (gr_line (start 98.5 70) (end 100 70) (layer Edge.Cuts) (width 0.05))
@@
   (gr_line (start 173 75) (end 161 81) (layer Edge.Cuts) (width 0.05))
   (gr_line (start 173 73.000001) (end 161 67) (layer Edge.Cuts) (width 0.05))
-  (gr_line (start 161 81) (end 100 81) (layer Edge.Cuts) (width 0.05))
+  (gr_line (start 161 81) (end 106.5 81) (layer Edge.Cuts) (width 0.05))
   (gr_line (start 100 67) (end 161 67) (layer Edge.Cuts) (width 0.05))
   (via (at 99.5 68) (size 0.8) (drill 0.4) (layers F.Cu B.Cu) (net 1))
@@
   (via (at 99.5 69) (size 0.8) (drill 0.4) (layers F.Cu B.Cu) (net 1))
   (via (at 100.5 69) (size 0.8) (drill 0.4) (layers F.Cu B.Cu) (net 1))
+  (via (at 100.5 82) (size 0.8) (drill 0.4) (layers F.Cu B.Cu) (net 2))
+  (via (at 99.5 82) (size 0.8) (drill 0.4) (layers F.Cu B.Cu) (net 2))
+  (via (at 100.5 81) (size 0.8) (drill 0.4) (layers F.Cu B.Cu) (net 2))
+  (via (at 99.5 81) (size 0.8) (drill 0.4) (layers F.Cu B.Cu) (net 2))
   (via (at 99.5 79) (size 0.8) (drill 0.4) (layers F.Cu B.Cu) (net 2))
   (via (at 99.5 80) (size 0.8) (drill 0.4) (layers F.Cu B.Cu) (net 2))
@@
     (polygon
       (pts
-        (xy 169 83) (xy 97 83) (xy 97 78) (xy 102 78) (xy 102 75)
-        (xy 169 75)
+        (xy 169 83) (xy 106.5 83) (xy 97 83) (xy 97 78.5) (xy 102.25 78.5)
+        (xy 102.25 75) (xy 169 75)
       )
     )
